Commit message: attaching to the gripper, peding rpy values

File: ros/handy_description/urdf/handy_description.urdf.xacro (robot description, xacro)
@@ -5,3 +5,8 @@
     filename="$(find finalarm_description)/urdf/finalarm_description.urdf.xacro"
   />
+    <xacro:arg name="use_default" default="false"/>
+    <xacro:arg name="parent" default="link_8"/>
+    <xacro:include
+    filename="$(find realsense2_custom_description)/urdf/d435_camera.urdf.xacro"
+  />
 </robot>

File: ros/realsense2_custom_description/urdf/d435_camera.urdf.xacro (robot description, xacro)
@@ -9,10 +9,14 @@
   <xacro:arg name="publish_pointcloud" default="false" />
   <xacro:arg name="gravity" default="1" />
+  <xacro:arg name="parent" default="base_link" />
+  <xacro:arg name="use_default" default="true"/>
   <xacro:include
     filename="$(find realsense2_custom_description)/urdf/_d435.urdf.xacro"
   />
-  <link name="base_link" />
+   <xacro:if value="$(arg use_default)">
+    <link name="base_link" />
+   </xacro:if>
   <xacro:sensor_d435
-    parent="base_link"
+    parent="$(arg parent)"
     use_nominal_extrinsics="$(arg use_nominal_extrinsics)"
     add_plug="$(arg add_plug)"
@@ -24,5 +28,5 @@
     gravity="$(arg gravity)"
   >
-    <origin xyz="0 0 0" rpy="0 0 0" />
+    <origin xyz="0 -0.015 -0.07" rpy="0 0 0" />
   </xacro:sensor_d435>
 </robot>
